File: splinter/KiCad/left.kicad_pcb (KiCad board)
At the start: 2 copper layers, 165.2 x 132.9 mm, 3 parts

Commit message: Add new pcb
Parts:
- removed MCU1: , ProMicro
- removed TRRS1: TRRS-PJ-320A-dual, TRRS-PJ-320A-dual
- added BotLeftM2: M2, MountingHole:MountingHole_2.2mm_M2, F.Cu at (59.5, 117.0)
- added BotRightM2: M2, MountingHole:MountingHole_2.2mm_M2, F.Cu at (179.0, 117.0)
- added D1: , ComboDiode, F.Cu at (45.2, 131.2)
- added D10: , ComboDiode, F.Cu at (69.0, 55.0)
- added D11: , ComboDiode, F.Cu at (88.1, 128.2)
- added D12: , ComboDiode, F.Cu at (88.1, 109.2)
- added D13: , ComboDiode, F.Cu at (88.1, 90.1)
- added D14: , ComboDiode, F.Cu at (88.1, 71.0)
- added D15: , ComboDiode, F.Cu at (88.1, 52.0)
- added D16: , ComboDiode, F.Cu at (107.2, 106.2)
- added D17: , ComboDiode, F.Cu at (107.2, 87.1)
- added D18: , ComboDiode, F.Cu at (107.2, 68.0)
- added D19: , ComboDiode, F.Cu at (107.2, 49.0)
- added D2: , ComboDiode, F.Cu at (45.2, 112.2)
- added D20: , ComboDiode, F.Cu at (126.2, 109.2)
- added D21: , ComboDiode, F.Cu at (126.2, 90.1)
- added D22: , ComboDiode, F.Cu at (126.2, 71.0)
- added D23: , ComboDiode, F.Cu at (126.2, 52.0)
- added D24: , ComboDiode, F.Cu at (145.2, 112.2)
- added D25: , ComboDiode, F.Cu at (145.2, 93.1)
- added D26: , ComboDiode, F.Cu at (145.2, 74.0)
- added D27: , ComboDiode, F.Cu at (145.2, 55.0)
- added D28: , ComboDiode, F.Cu at (145.9, 136.0)
- added D29: , ComboDiode, F.Cu at (172.6, 145.9)
- added D3: , ComboDiode, F.Cu at (45.2, 93.1)
- added D4: , ComboDiode, F.Cu at (45.2, 74.0)
- added D5: , ComboDiode, F.Cu at (50.0, 55.0)
- added D6: , ComboDiode, F.Cu at (69.0, 131.2)
- added D7: , ComboDiode, F.Cu at (69.0, 112.2)
- added D8: , ComboDiode, F.Cu at (69.0, 93.1)
- added D9: , ComboDiode, F.Cu at (69.0, 74.0)
- added LeftM3: M3, MountingHole:MountingHole_3.2mm_M3, F.Cu at (56.0, 89.0)
- added LeftM3: M3, MountingHole:MountingHole_3.2mm_M3, F.Cu at (165.0, 89.0)
- added S1: , MX, F.Cu at (45.2, 126.2)
- added S10: , MX, F.Cu at (69.0, 50.0)
- added S11: , MX, F.Cu at (88.1, 123.2)
- added S12: , MX, F.Cu at (88.1, 104.2)
- added S13: , MX, F.Cu at (88.1, 85.1)
- added S14: , MX, F.Cu at (88.1, 66.0)
- added S15: , MX, F.Cu at (88.1, 47.0)
- added S16: , MX, F.Cu at (107.2, 101.2)
- added S17: , MX, F.Cu at (107.2, 82.1)
- added S18: , MX, F.Cu at (107.2, 63.0)
- added S19: , MX, F.Cu at (107.2, 44.0)
- added S2: , MX, F.Cu at (45.2, 107.2)
- added S20: , MX, F.Cu at (126.2, 104.2)
- added S21: , MX, F.Cu at (126.2, 85.1)
- added S22: , MX, F.Cu at (126.2, 66.0)
- added S23: , MX, F.Cu at (126.2, 47.0)
- added S24: , MX, F.Cu at (145.2, 107.2)
- added S25: , MX, F.Cu at (145.2, 88.1)
- added S26: , MX, F.Cu at (145.2, 69.0)
- added S27: , MX, F.Cu at (145.2, 50.0)
- added S28: , MX, F.Cu at (147.2, 131.2)
- added S29: , MX, F.Cu at (174.7, 141.3)
- added S3: , MX, F.Cu at (45.2, 88.1)
- added S4: , MX, F.Cu at (45.2, 69.0)
- added S5: , MX, F.Cu at (50.0, 50.0)
- added S6: , MX, F.Cu at (69.0, 126.2)
- added S7: , MX, F.Cu at (69.0, 107.2)
- added S8: , MX, F.Cu at (69.0, 88.1)
- added S9: , MX, F.Cu at (69.0, 69.0)
- added TRRS: TRRS-PJ-320A-dual, TRRS-PJ-320A-dual, B.Cu at (178.0, 33.0)
- added TopLeftM2: M2, MountingHole:MountingHole_2.2mm_M2, F.Cu at (59.5, 60.0)
- added TopRightM2: M2, MountingHole:MountingHole_2.2mm_M2, F.Cu at (179.0, 60.0)
- added atmega32u4: , ProMicro, B.Cu at (165.0, 50.4)
- Reset button: renamed from B1; moved to B.Cu
- moved Reset button 221.2 mm to (165.0, 75.0), turned to 180 degrees
Connections:
- Reset button pad 1: RST -> GND
- Reset button pad 2: GND -> RST
Routing:
- net P7: track 0.00 -> 289.7 mm
- net P15: track 0.00 -> 262.9 mm
- net P8: track 0.00 -> 252.1 mm
- net P18: track 0.00 -> 216.3 mm
- net P9: track 0.00 -> 209.4 mm
- net P19: track 0.00 -> 201.5 mm
- net P14: track 0.00 -> 197.3 mm, vias 0 -> 1
- net P20: track 0.00 -> 185.5 mm
- net P10: track 0.00 -> 176.4 mm
- net P21: track 0.00 -> 165.4 mm
- net P16: track 0.00 -> 147.0 mm, vias 0 -> 1
- net GND: track 0.00 -> 51.4 mm
- net RST: track 0.00 -> 38.9 mm
- net VCC: track 0.00 -> 25.9 mm
- net mod_meta: track 0.00 -> 16.1 mm
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Other:
- board size 165.2 x 132.9 mm -> 149 x 119 mm
- net class Default removed
- board text added: "{dblquote}Splinter{dblquote} 61-key split columnar keyboard by Andornaut"
