File: kicad/left.kicad_pcb (KiCad board)
At the start: 2 copper layers, 155.5 x 119.1 mm, 61 parts

Commit message: Iterate on PCB and new case
Routing:
- net P20: track 148.5 -> 145.4 mm
Changed lines of the file:
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@@
   (segment (start 233.56754 202.85) (end 233.56754 202.73246) (width 0.25) (layer "F.Cu") (net 1))
   (via (at 230.113863 206.313156) (size 0.8) (drill 0.4) (layers "F.Cu" "B.Cu") (remove_unused_layers) (keep_end_layers) (free) (zone_layer_connections) (net 1))
-  (segment (start 213.127208 210.9) (end 206.377208 204.15) (width 0.25) (layer "B.Cu") (net 1))
-  (segment (start 133.04 198.14) (end 119.5 184.6) (width 0.25) (layer "B.Cu") (net 1))
-  (segment (start 230.104384 206.313156) (end 225.51754 210.9) (width 0.25) (layer "B.Cu") (net 1))
   (segment (start 109.6775 155.56) (end 109.6775 136.51) (width 0.25) (layer "B.Cu") (net 1))
+  (segment (start 109.8 184.4) (end 109.7 184.5) (width 0.25) (layer "B.Cu") (net 1))
+  (segment (start 224.814413 210.9) (end 224.764413 210.95) (width 0.25) (layer "B.Cu") (net 1))
+  (segment (start 132.99 203.907107) (end 132.99 198.09) (width 0.25) (layer "B.Cu") (net 1))
+  (segment (start 109.6775 131.7225) (end 109.6775 136.51) (width 0.25) (layer "B.Cu") (net 1))
+  (segment (start 206.356498 204.2) (end 133.282893 204.2) (width 0.25) (layer "B.Cu") (net 1))
+  (segment (start 119.3 184.4) (end 109.8 184.4) (width 0.25) (layer "B.Cu") (net 1))
   (segment (start 230.113863 206.313156) (end 230.104384 206.313156) (width 0.25) (layer "B.Cu") (net 1))
-  (segment (start 109.6775 131.7225) (end 109.6775 136.51) (width 0.25) (layer "B.Cu") (net 1))
-  (segment (start 225.51754 210.9) (end 213.127208 210.9) (width 0.25) (layer "B.Cu") (net 1))
-  (segment (start 133.04 204.16) (end 133.04 198.14) (width 0.25) (layer "B.Cu") (net 1))
-  (segment (start 206.377208 204.15) (end 133.05 204.15) (width 0.25) (layer "B.Cu") (net 1))
+  (segment (start 133.282893 204.2) (end 132.99 203.907107) (width 0.25) (layer "B.Cu") (net 1))
+  (segment (start 109.7 184.5) (end 109.7 184.6) (width 0.25) (layer "B.Cu") (net 1))
   (segment (start 114.44 126.96) (end 109.6775 131.7225) (width 0.25) (layer "B.Cu") (net 1))
-  (segment (start 133.05 204.15) (end 133.04 204.16) (width 0.25) (layer "B.Cu") (net 1))
-  (segment (start 119.5 184.6) (end 109.7 184.6) (width 0.25) (layer "B.Cu") (net 1))
+  (segment (start 225.51754 210.9) (end 224.814413 210.9) (width 0.25) (layer "B.Cu") (net 1))
   (segment (start 109.7 184.6) (end 109.7 193.6375) (width 0.25) (layer "B.Cu") (net 1))
+  (segment (start 132.99 198.09) (end 119.3 184.4) (width 0.25) (layer "B.Cu") (net 1))
   (segment (start 109.6775 155.56) (end 109.6775 174.61) (width 0.25) (layer "B.Cu") (net 1))
   (segment (start 114.44 118.16) (end 114.44 126.96) (width 0.25) (layer "B.Cu") (net 1))
   (segment (start 109.7 174.6325) (end 109.7 184.6) (width 0.25) (layer "B.Cu") (net 1))
+  (segment (start 224.764413 210.95) (end 213.106498 210.95) (width 0.25) (layer "B.Cu") (net 1))
+  (segment (start 230.104384 206.313156) (end 225.51754 210.9) (width 0.25) (layer "B.Cu") (net 1))
+  (segment (start 213.106498 210.95) (end 206.356498 204.2) (width 0.25) (layer "B.Cu") (net 1))
   (segment (start 120.4 201.2) (end 123.8 197.8) (width 0.25) (layer "B.Cu") (net 2))
   (segment (start 123.8 192.3155) (end 122.6045 191.12) (width 0.25) (layer "B.Cu") (net 2))
@@
   (segment (start 247 133.32) (end 244.445 133.32) (width 0.25) (layer "F.Cu") (net 13))
   (via (at 228.700353 204.899646) (size 0.8) (drill 0.4) (layers "F.Cu" "B.Cu") (remove_unused_layers) (keep_end_layers) (free) (zone_layer_connections) (net 13))
+  (segment (start 152.54 185.84) (end 152.54 185.7) (width 0.25) (layer "B.Cu") (net 13))
+  (segment (start 184 203.2) (end 166.7 185.9) (width 0.25) (layer "B.Cu") (net 13))
+  (segment (start 213.52071 209.95) (end 206.77071 203.2) (width 0.25) (layer "B.Cu") (net 13))
   (segment (start 152.54 171.61) (end 152.54 152.56) (width 0.25) (layer "B.Cu") (net 13))
-  (segment (start 228.700353 204.899646) (end 223.599999 210) (width 0.25) (layer "B.Cu") (net 13))
-  (segment (start 223.599999 210) (end 213.5 210) (width 0.25) (layer "B.Cu") (net 13))
-  (segment (start 189.2 185.7) (end 152.54 185.7) (width 0.25) (layer "B.Cu") (net 13))
-  (segment (start 213.5 210) (end 189.2 185.7) (width 0.25) (layer "B.Cu") (net 13))
+  (segment (start 228.700353 204.899646) (end 223.649999 209.95) (width 0.25) (layer "B.Cu") (net 13))
+  (segment (start 206.77071 203.2) (end 184 203.2) (width 0.25) (layer "B.Cu") (net 13))
+  (segment (start 152.6 185.9) (end 152.54 185.84) (width 0.25) (layer "B.Cu") (net 13))
+  (segment (start 166.7 185.9) (end 152.6 185.9) (width 0.25) (layer "B.Cu") (net 13))
   (segment (start 152.54 190.66) (end 152.54 171.61) (width 0.25) (layer "B.Cu") (net 13))
+  (segment (start 223.649999 209.95) (end 213.52071 209.95) (width 0.25) (layer "B.Cu") (net 13))
   (segment (start 152.54 114.46) (end 152.54 133.51) (width 0.25) (layer "B.Cu") (net 13))
   (segment (start 152.54 152.56) (end 152.54 133.51) (width 0.25) (layer "B.Cu") (net 13))
@@
   (segment (start 182.5 119) (end 180.488684 119) (width 0.25) (layer "B.Cu") (net 23))
   (segment (start 185.7 110.103) (end 185.7 115.8) (width 0.25) (layer "B.Cu") (net 23))
-  (segment (start 190.64 186.503604) (end 201.049211 196.912815) (width 0.25) (layer "B.Cu") (net 24))
   (segment (start 190.64 114.46) (end 190.64 133.51) (width 0.25) (layer "B.Cu") (net 24))
+  (segment (start 190.64 171.61) (end 190.64 181.24) (width 0.25) (layer "B.Cu") (net 24))
+  (segment (start 206.312815 196.912815) (end 212.386776 196.912815) (width 0.25) (layer "B.Cu") (net 24))
   (segment (start 205.031802 109.45) (end 208.081802 112.5) (width 0.25) (layer "B.Cu") (net 24))
   (segment (start 225.4 118.1) (end 229.185 118.1) (width 0.25) (layer "B.Cu") (net 24))
   (segment (start 190.64 152.56) (end 190.64 133.51) (width 0.25) (layer "B.Cu") (net 24))
   (segment (start 190.64 114.46) (end 190.64 109.45) (width 0.25) (layer "B.Cu") (net 24))
-  (segment (start 190.64 171.61) (end 190.64 186.503604) (width 0.25) (layer "B.Cu") (net 24))
+  (segment (start 190.64 181.24) (end 206.312815 196.912815) (width 0.25) (layer "B.Cu") (net 24))
   (segment (start 190.64 109.45) (end 205.031802 109.45) (width 0.25) (layer "B.Cu") (net 24))
   (segment (start 208.081802 112.5) (end 225.4 112.5) (width 0.25) (layer "B.Cu") (net 24))
-  (segment (start 201.049211 196.912815) (end 212.386776 196.912815) (width 0.25) (layer "B.Cu") (net 24))
   (segment (start 225.4 112.5) (end 225.4 118.1) (width 0.25) (layer "B.Cu") (net 24))
   (segment (start 190.64 152.56) (end 190.64 171.61) (width 0.25) (layer "B.Cu") (net 24))
