File: v4/kicad/right.kicad_pcb (KiCad board)
At the start: 2 copper layers, 158.5 x 119.3 mm, 70 parts

Commit message: Place v4 TRRS data-line protection and update footprints
Add the SMF3.3CA TVS (sod-123fl) and 100Ohm 0805 series resistor
(infused-kim/smd_0805) below the TRRS jack on side B, mirrored to the
right half, and regenerate the kicad PCBs with the new components.
Replace the old placeholder resistor_0603/sod-323 footprints and add
the resistor and TVS BOM entries.
Parts:
- added D33: SOD-123FL, Diode_SMD:D_SOD-123FL, F.Cu at (228.1, 114.5)
- added SMD1: , smd_805, F.Cu at (228.1, 117.5)
Connections:
- TRRS1 pad 2: P0 -> DATA_RAW

Commit message: Fix custom diode footprint attributes and sod-123fl geometry
After auditing the custom footprints against manufacturer outline drawings:
- sod-123fl, sod-123w: change (attr smd) to (attr through_hole) to match
  the actual reversible hand-solder pads (resolves the SMD-vs-THT DRC/BOM
  mismatch).
- sod-123fl: widen pads to 1.1x1.35mm for proper side fillets, widen the
  courtyard to +/-2.45mm (0.25mm pad clearance), move the silkscreen body
  lines out of the pads, and rename from the nonexistent stock name
  Diode_SMD:D_SOD-123FL to splinter:D_SOD-123FL_HandSolder.
Re-sync the regenerated footprints into the unrouted v4/kicad boards.
mcu_liatris pinout and geometry verified correct (incl. against hardware);
no change needed.
Parts:
- D33: footprint Diode_SMD:D_SOD-123FL -> splinter:D_SOD-123FL_HandSolder
